File: untitled.sch (EAGLE design)
At the start: 7 parts, among them IC1 L293D, IC2 L293D

Commit message: pcb finished
Parts:
- added JP10, JP11, JP12, JP14: (no value), pinhead:PINHD-1X3
- added JP13, JP15, JP5, JP7, JP9: PINHD-1X4, Connector:PINHD-1X4
- added JP6, JP8: PINHD-1X2, Connector:PINHD-1X2
- added R1, R10, R11, R12, R2, R3, R4, R5, R6, R7, R8, R9: (no value), adafruit:R-US_0204/2V
- added T1, T2, T3, T4: 2N2222, adafruit:2N2222
Connections:
- new net AVATAR_RX: JP9.2, U$1.PB3(D13)
- new net AVATAR_TX: JP9.1, U$1.PB4(D12)
- new net EN: IC1.1-2EN, IC1.3-4EN, IC2.1-2EN, IC2.3-4EN, U$1.PA5(A4)
- new net ENC_A_1: JP2.2, U$1.PA0(A0)
- new net ENC_A_2: JP1.2, U$1.PF1(D8)
- new net ENC_A_3: JP5.2, U$1.PA11(D10)
- new net ENC_A_4: JP7.2, U$1.PA12(D2)
- new net ENC_B_1: JP2.3, U$1.PB1(D6)
- new net ENC_B_2: JP1.3, U$1.PA8(D9)
- new net ENC_B_3: JP5.3, U$1.PB5(D11)
- new net ENC_B_4: JP7.3, U$1.PA2(A7)
- new net GM1: JP10.1, U$1.PF0(D7)
- new net GM2: JP11.1, U$1.PB0(D3)
- new net GM3: JP14.1, U$1.PA1(A1)
- new net GND: IC1.GND1, IC1.GND2, IC1.GND3, IC1.GND4, IC2.GND1, IC2.GND2, IC2.GND3, IC2.GND4, JP1.4, JP10.3, JP11.3, JP12.3, JP13.4, JP14.3, JP15.4, JP2.4, JP5.4, JP7.4, JP9.4, R11.2, R2.2, R5.2, R8.2, T1.E, T2.E, T3.E, T4.E, U$1.GND@1, U$1.GND@2
- new net I²C_SCL: JP15.1, U$1.PB6(D5)
- new net I²C_SDA: JP15.2, U$1.PB7(D4)
- new net M1: IC1.1A, R1.1, U$1.PA3(A2)
- new net M1N: IC1.2A, R3.1, T1.C
- new net M2: IC1.4A, R4.1, U$1.PA4(A3)
- new net M2N: IC1.3A, R6.1, T2.C
- new net M3: IC2.1A, R7.1, U$1.PA6(A5)
- new net M3N: IC2.2A, R9.1, T3.C
- new net M4: IC2.4A, R10.1, U$1.PA7(A6)
- new net M4N: IC2.3A, R12.1, T4.C
- new net N$10: IC2.3Y, JP8.1
- new net N$11: IC2.4Y, JP8.2
- new net N$14: R1.2, R2.1, T1.B
- new net N$15: R4.2, R5.1, T2.B
- new net N$19: R7.2, R8.1, T3.B
- new net N$22: R10.2, R11.1, T4.B
- new net N$4: IC1.4Y, JP3.2
- new net N$5: IC1.3Y, JP3.1
- new net N$6: IC1.2Y, JP4.2
- new net N$7: IC1.1Y, JP4.1
- new net N$8: IC2.1Y, JP6.1
- new net N$9: IC2.2Y, JP6.2
- new net TBS_RX: JP13.1, U$1.PA9(D1/TX)
- new net TBS_TX: JP13.2, U$1.PA10(D0/RX)
- net 3V3: now also R12.2, R3.2, R6.2, R9.2
- net 5V0: now also IC1.VCC1, IC2.VCC1, JP1.1, JP10.2, JP11.2, JP12.1, JP13.3, JP14.2, JP15.3, JP2.1, JP5.1, JP7.1
- net 9V0: now also IC1.VCC2, IC2.VCC2, JP12.2, JP9.3
Other:
- moved on the sheet: JP1, JP2, JP3, JP4, U$1
